Commit message: add depth camera and fix camera&imu display

File: src/Mid360_simulation_plugin/livox_laser_simulation/models/car_model.xacro (robot description, xacro)
@@ -27,5 +27,5 @@
             </geometry>
         </collision>
-        <xacro:inertial_matrix mass="1"/>
+        <xacro:inertial_matrix mass="10"/>
 		<kinematic>1</kinematic>
 		<gravity>9.8</gravity>

File: src/Mid360_simulation_plugin/livox_laser_simulation/models/cyBlackPearl.xacro (robot description, xacro)
@@ -4,6 +4,8 @@
   <xacro:include filename="$(find livox_laser_simulation)/models/car_model.xacro" />
   <xacro:include filename="$(find livox_laser_simulation)/models/imu.xacro" />
+  <xacro:include filename="$(find livox_laser_simulation)/models/camera.xacro" />
   <xacro:Livox_Mid360 name="livox" />
   <xacro:imu_sensor name="imu" />
   <xacro:link_oasis name="oasis" />
+  <xacro:camera_sensor name="camera" />
 </robot>

File: src/Mid360_simulation_plugin/livox_laser_simulation/models/imu.xacro (robot description, xacro)
@@ -33,8 +33,8 @@
   </xacro:macro>
   <xacro:macro name="imu_sensor" params="name:=imu parentLink:=oasis_300">
-    <link name="${name}" />
+    <link name="${name}">
     <xacro:IMU_inertial_matrix />
     <visual>
-      <origin xyz="-0.35 0 0.03" rpy="0 0 0" />
+      <origin xyz="0 0 0" rpy="0 0 0" />
       <geometry>
         <box size="0.1 0.07 0.03" />
@@ -45,6 +45,7 @@
         <box size="0.1 0.07 0.03" />
       </geometry>
-      <origin xyz="0 0 0" rpy="0 0 0" />
+      <origin xyz="0.0 0 0.0" rpy="0 0 0" />
     </collision>
+    </link>
     <joint name="imu2oasis_300" type="fixed">
       <parent link="${parentLink}" />
@@ -52,6 +53,7 @@
       <origin xyz="-0.35 0 0.03" />
     </joint>
-    <xacro:gazebo_ros_imu TopicName="livox/imu" name="imu"/>
+    <xacro:gazebo_ros_imu TopicName="livox/imu" name="imu" />
   </xacro:macro>
-  <!--xacro:imu_sensor name="imu" /-->
+  <!--xacro:imu_sensor
+  name="imu" /-->
 </robot>

File: src/Mid360_simulation_plugin/livox_laser_simulation/models/livox_mid360.xacro (robot description, xacro)
@@ -21,5 +21,5 @@
    <!-- This is laser plugin macro -->
   <xacro:macro name="Livox_Mid_gazebo_sensor"
-    params="visualize:=True update_rate:=10 resolution:=0.002 noise_mean:=0.0 noise_stddev:=0.01 name:=livox">
+    params="visualize:=true update_rate:=10 resolution:=0.002 noise_mean:=0.0 noise_stddev:=0.01 name:=livox">
     <gazebo reference="${name}">
       <sensor type="ray" name="laser_${name}">
@@ -63,5 +63,5 @@
           <!--csv_file_name>package://livox_laser_simulation/scan_mode/mid360-real-centr.csv</csv_file_name-->
           <csv_file_name>mid360-real-centr.csv</csv_file_name>
-          <publish_pointcloud_type>3</publish_pointcloud_type>
+          <publish_pointcloud_type>2</publish_pointcloud_type>
           <ros_topic>${ros_topic}</ros_topic>
           <frameName>livox</frameName>
@@ -71,5 +71,5 @@
   </xacro:macro>
 <!-- This is Mid360 Plugin macro which integrate the gazebo laser plugin-->
-  <xacro:macro name="Livox_Mid360" params="visualize:=True name:=livox">
+  <xacro:macro name="Livox_Mid360" params="visualize:=true name:=livox">
     <!-- This is Mid360 mesh -->>
     <link name="${name}_base">
