Commit message: finish cyBlackPearl sim with multisensor

File: src/carurdf/urdf/carurdf.urdf (robot description, URDF)
Before this commit: robot carurdf, 5 links, 4 joints
Links:
- added link base_footprint; visual sphere radius=0.001
- added link camera
- added link imu; visual box size=0.01 0.01 0.01
- added link mid360; visual box size=0.01 0.01 0.01
- added link multisensor; visual mesh filename=package://carurdf/meshes/multisensor.dae
- link base_link: mass 246.126252736902 -> 1.6126252736902
- link wheel11: mass 1.2166 -> 0.12166
- link wheel12: mass 1.2166 -> 0.12166
- link wheel21: mass 1.2166 -> 0.12166
- link wheel22: mass 1.2166 -> 0.12166
Joints:
- added joint base2multisensor: type fixed, parent base_link, child multisensor, origin xyz=0.459805472903942 0 0.07482260358453 rpy=0 0 0
- added joint base_footprint2base_link: type fixed, parent base_footprint, child base_link, origin xyz=0 0 0.001  rpy=0 0 0
- added joint camera2multisensor: type fixed, parent multisensor, child camera, origin xyz=0.117 -0.052355 0 rpy=0 0 0
- added joint imu2multisensor: type fixed, parent multisensor, child imu, origin xyz=0.0117 0 0
- added joint lidar2multisensor: type fixed, parent multisensor, child mid360, origin xyz=0.0117 0.052355 0 rpy=0 0 -0.7853
